Commit message: paolo changed tez_workcell to tez_description

File: tez_description/urdf/tez_cell_boxes.urdf (robot description, URDF)
Before this commit: robot tez_cell, 17 links, 16 joints
Links:
- link jig: geometry collision mesh filename=package://tez_description/mesh/reduced_details/jig.dae; visual mesh filename=package://tez_description/mesh/reduced_details/jig.dae
- link linear_axis: geometry collision mesh filename=package://tez_description/mesh/full_details/linear_axis.dae; visual mesh filename=package://tez_description/mesh/full_details/linear_axis.dae

File: tez_description/urdf/tez_cell_reducedmesh.urdf (robot description, URDF)
Before this commit: robot tez_cell, 17 links, 16 joints
Links:
- link KR210_1_A1: geometry collision mesh filename=package://tez_description/mesh/reduced_details/KR210_3100_u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; visual mesh filename=package://tez_description/mesh/reduced_details/KR210_3100_u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
- link KR210_1_A2: geometry collision mesh filename=package://tez_description/mesh/reduced_details/KR210_3100_u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; visual mesh filename=package://tez_description/mesh/reduced_details/KR210_3100_u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
- link KR210_1_A3: geometry collision mesh filename=package://tez_description/mesh/reduced_details/KR210_3100_u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; visual mesh filename=package://tez_description/mesh/reduced_details/KR210_3100_u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
- link KR210_1_A4: geometry collision mesh filename=package://tez_description/mesh/reduced_details/KR210_3100_u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; visual mesh filename=package://tez_description/mesh/reduced_details/KR210_3100_u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
- link KR210_1_A5: geometry collision mesh filename=package://tez_description/mesh/reduced_details/KR210_3100_u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; visual mesh filename=package://tez_description/mesh/reduced_details/KR210_3100_u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
- link KR210_1_A6: geometry collision mesh filename=package://tez_description/mesh/reduced_details/KR210_3100_u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; visual mesh filename=package://tez_description/mesh/reduced_details/KR210_3100_u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
- link KR210_1_socket: geometry collision mesh filename=package://tez_description/mesh/reduced_details/KR210_3100_u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; visual mesh filename=package://tez_description/mesh/reduced_details/KR210_3100_u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
- link KR210_2_A1: geometry collision mesh filename=package://tez_description/mesh/reduced_details/KR210_3100_u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; visual mesh filename=package://tez_description/mesh/reduced_details/KR210_3100_u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
- link KR210_2_A2: geometry collision mesh filename=package://tez_description/mesh/reduced_details/KR210_3100_u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; visual mesh filename=package://tez_description/mesh/reduced_details/KR210_3100_u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
- link KR210_2_A3: geometry collision mesh filename=package://tez_description/mesh/reduced_details/KR210_3100_u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; visual mesh filename=package://tez_description/mesh/reduced_details/KR210_3100_u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
- link KR210_2_A4: geometry collision mesh filename=package://tez_description/mesh/reduced_details/KR210_3100_u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; visual mesh filename=package://tez_description/mesh/reduced_details/KR210_3100_u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
- link KR210_2_A5: geometry collision mesh filename=package://tez_description/mesh/reduced_details/KR210_3100_u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; visual mesh filename=package://tez_description/mesh/reduced_details/KR210_3100_u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
- link KR210_2_A6: geometry collision mesh filename=package://tez_description/mesh/reduced_details/KR210_3100_u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; visual mesh filename=package://tez_description/mesh/reduced_details/KR210_3100_u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
- link KR210_2_socket: geometry collision mesh filename=package://tez_description/mesh/reduced_details/KR210_3100_u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; visual mesh filename=package://tez_description/mesh/reduced_details/KR210_3100_u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
- link base_link: geometry collision mesh filename=package://tez_description/mesh/reduced_details/spannfeld.dae; visual mesh filename=package://tez_description/mesh/reduced_details/spannfeld.dae
- link jig: geometry collision mesh filename=package://tez_description/mesh/reduced_details/jig.dae; visual mesh filename=package://tez_description/mesh/reduced_details/jig.dae
- link linear_axis: geometry collision mesh filename=package://tez_description/mesh/reduced_details/linear_axis.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; visual mesh filename=package://tez_description/mesh/reduced_details/linear_axis.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
