Commit message: paolo: tez two robots

File: tez_description/urdf/tez_cell_reducedmesh.urdf (robot description, URDF)
Before this commit: robot tez_cell, 16 links, 15 joints
Links:
- added link gripper; collision mesh filename=package://tez_description/mesh/collada/reduced_details/grip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; visual mesh filename=package://tez_description/mesh/collada/reduced_details/grip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
Joints:
- added joint EndEffector: type fixed, parent KR210_2_A6, child gripper, origin xyz=0 -0.01 0 rpy=0 0 1.5708, axis 0 0 0
- joint kr210_1_joint_1: limit lower=-3.22886 upper=3.22886 effort=100 velocity=1 -> lower=-3.22886 upper=3.22886 effort=100 velocity=0.1
- joint kr210_1_joint_2: limit lower=-2.443460952792061 upper=-0.08726646259971647 effort=10000 velocity=1 -> lower=-2.443460952792061 upper=-0.08726646259971647 effort=10000 velocity=0.1
- joint kr210_1_joint_3: limit lower=-2.0943951023931953 upper=2.705260340591211 effort=100 velocity=1 -> lower=-2.0943951023931953 upper=2.705260340591211 effort=100 velocity=0.1
- joint kr210_1_joint_5: limit lower=-2.138028333693054 upper=2.138028333693054 effort=100 velocity=1 -> lower=-2.138028333693054 upper=2.138028333693054 effort=100 velocity=0.1
- joint kr210_2_joint_1: axis 0.0 0.0 1.0 -> 0.0 0.0 -1.0; limit lower=-3.22886 upper=3.22886 effort=100 velocity=100 -> lower=-3.22886 upper=3.22886 effort=100 velocity=0.1; origin xyz=0 0 0.5256 rpy=0 0 0 -> xyz=0 0 0.5256 rpy=0 0 -1.5707963267948966
- joint kr210_2_joint_2: limit lower=-2.0944 upper=1.22173 effort=10000 velocity=100 -> lower=-2.443460952792061 upper=-0.08726646259971647 effort=10000 velocity=0.1; origin xyz=0.005 -0.35 0.45 rpy=0 0 0 -> xyz=0.005 -0.35 0.45 rpy=1.5707963267948966 0 0
- joint kr210_2_joint_3: limit lower=-2.0944 upper=2.70526 effort=100 velocity=100 -> lower=-2.0943951023931953 upper=2.705260340591211 effort=100 velocity=0.1; origin xyz=-0.183 0 1.35 rpy=0 0 0 -> xyz=-0.183 0 1.35 rpy=-1.5707963267948966 0 0
- joint kr210_2_joint_5: limit lower=-2.18166 upper=2.18166 effort=100 velocity=100 -> lower=-2.138028333693054 upper=2.138028333693054 effort=100 velocity=0.1
- joint kr210_2_linear_axis_joint: limit lower=1.5 upper=9 effort=100 velocity=100 -> lower=-9 upper=0 effort=100 velocity=100; origin xyz=-1.5 0 0.487 rpy=0 0 3.14159 -> xyz=-9.0 0 0.487 rpy=0 0 3.1415
